Commit message: a

File: src/bumperbot_description/urdf/bumperbot.xacro (robot description, xacro)
@@ -1,5 +1,7 @@
 <?xml version="1.0"?>
 <robot name="bumperbot" xmlns:xacro="http://ros.org/wiki/xacro">
+  <!-- Base Footprint Link -->
   <link name="base_footprint"/>
+  <!-- Base Link -->
   <link name="base_link">
     <visual>
@@ -9,5 +11,16 @@
       </geometry>
     </visual>
+    <collision>
+      <origin xyz="0 0 0" rpy="0 0 0"/>
+      <geometry>
+        <mesh filename="package://bumperbot_description/meshes/sasi.STL" scale="0.001 0.001 0.001"/>
+      </geometry>
+    </collision>
+    <inertial>
+      <mass value="5.0"/>
+      <inertia ixx="0.1" ixy="0" ixz="0" iyy="0.1" iyz="0" izz="0.1"/>
+    </inertial>
   </link>
+  <!-- Base Joint -->
   <joint name="base_joint" type="fixed">
     <parent link="base_footprint"/>
@@ -15,24 +28,31 @@
     <origin xyz="0 0 0.033" rpy="0 0 0"/>
   </joint>
-<link name="wheel_right_link">
-  <visual>
-    <!-- STL'nin link merkezine göre hizalanması (robot konumu değil) -->
-    <origin xyz="0 -0.014 0" rpy="1.5708 0 0"/>
-    <geometry>
-      <!-- Sağ tekerin 3D modeli -->
-      <mesh filename="package://bumperbot_description/meshes/wheel_right_link.STL"/>
-    </geometry>
-  </visual>
-</link>
-<joint name="wheel_right_joint" type="continuous">
-  <!-- Tekerin bağlı olduğu ana gövde -->
-  <parent link="base_link"/>
-  <!-- Bu joint'in hareket ettirdiği parça -->
-  <child link="wheel_right_link"/>
-  <!-- Tekerin döndüğü eksen (Y ekseni) -->
-  <axis xyz="0 1 0"/>
-  <!-- Tekerin base_link'e göre robot üzerindeki konumu -->
-  <origin xyz="0 -0.07011 0" rpy="0 0 0"/>
-</joint>
+  <!-- Right Wheel -->
+  <link name="wheel_right_link">
+    <visual>
+      <origin xyz="0 -0.014 0" rpy="1.5708 0 0"/>
+      <geometry>
+        <mesh filename="package://bumperbot_description/meshes/wheel_right_link.STL"/>
+      </geometry>
+    </visual>
+    <collision>
+      <origin xyz="0 -0.014 0" rpy="1.5708 0 0"/>
+      <geometry>
+        <mesh filename="package://bumperbot_description/meshes/wheel_right_link.STL"/>
+      </geometry>
+    </collision>
+    <inertial>
+      <mass value="1.0"/>
+      <inertia ixx="0.01" ixy="0" ixz="0" iyy="0.01" iyz="0" izz="0.01"/>
+    </inertial>
+  </link>
+  <!-- Right Wheel Joint -->
+  <joint name="wheel_right_joint" type="continuous">
+    <parent link="base_link"/>
+    <child link="wheel_right_link"/>
+    <axis xyz="0 1 0"/>
+    <origin xyz="0 -0.07011 0" rpy="0 0 0"/>
+  </joint>
+  <!-- Left Wheel -->
   <link name="wheel_left_link">
     <visual>
@@ -42,11 +62,23 @@
       </geometry>
     </visual>
+    <collision>
+      <origin xyz="0 0.014 0" rpy="1.5708 0 3.1416"/>
+      <geometry>
+        <mesh filename="package://bumperbot_description/meshes/wheel_left_link.STL"/>
+      </geometry>
+    </collision>
+    <inertial>
+      <mass value="1.0"/>
+      <inertia ixx="0.01" ixy="0" ixz="0" iyy="0.01" iyz="0" izz="0.01"/>
+    </inertial>
   </link>
+  <!-- Left Wheel Joint -->
   <joint name="wheel_left_joint" type="continuous">
     <parent link="base_link"/>
     <child link="wheel_left_link"/>
     <axis xyz="0 1 0"/>
-    <origin xyz="0 0.0701101849418637 0" rpy="0 0 0"/>
+    <origin xyz="0 0.07011 0" rpy="0 0 0"/>
   </joint>
+  <!-- Caster Wheel -->
   <link name="caster_wheel_link">
     <visual>
@@ -56,5 +88,16 @@
       </geometry>
     </visual>
+    <collision>
+      <origin xyz="0 0 0" rpy="0 0 0"/>
+      <geometry>
+        <box size="0.03215 0.043575 0.035122"/> <!-- Caster tekerleği boyutlarına göre kutu geometrisi -->
+      </geometry>
+    </collision>
+    <inertial>
+      <mass value="0.00766"/> <!-- Kütle 7.66 g = 0.00766 kg -->
+      <inertia ixx="0.1456842" ixy="-0.004499" ixz="-0.007876" iyy="0.1154946" iyz="-0.0382781" izz="0.0921484"/>
+    </inertial>
   </link>
+  <!-- Caster Wheel Joint -->
   <joint name="caster_wheel_joint" type="fixed">
     <parent link="base_link"/>
