Commit message: urdf

File: install/bumperbot_description/share/bumperbot_description/urdf/bumperbot.xacro (robot description, xacro)
@@ -1,73 +1,59 @@
 <?xml version="1.0"?>
 <robot name="bumperbot" xmlns:xacro="http://ros.org/wiki/xacro">
-    <link name="base_footprint"/>
-    <link name="base_link">
-        <visual>
-            <origin xyz="0 0 0" rpy="0 0 0"/>
-            <geometry>
-                <mesh filename="package://bumperbot_description/meshes/sasi.STL" scale="0.001 0.001 0.001"/>
-            </geometry>
-        </visual>
-    </link>
-    <joint name="base_joint" type="fixed">
-        <parent link="base_footprint"/>
-        <child link="base_link"/>
-        <origin xyz="0 0 0" rpy="0 0 0.033"/>
-    </joint>
+  <link name="base_footprint"/>
+  <link name="base_link">
+    <visual>
+      <origin xyz="0 0 0" rpy="0 0 0"/>
+      <geometry>
+        <mesh filename="package://bumperbot_description/meshes/sasi.STL" scale="0.001 0.001 0.001"/>
+      </geometry>
+    </visual>
+  </link>
+  <joint name="base_joint" type="fixed">
+    <parent link="base_footprint"/>
+    <child link="base_link"/>
+    <origin xyz="0 0 0.033" rpy="0 0 0"/>
+  </joint>
   <link name="wheel_right_link">
     <visual>
-      <origin xyz="0 0 0" rpy="1.57 0 0" />
+      <origin xyz="0 -0.014 0" rpy="1.5708 0 0"/>
       <geometry>
-        <mesh filename="package://bumperbot_description/meshes/wheel_right_link.STL" scale="0.001 0.001 0.001"/>
+        <mesh filename="package://bumperbot_description/meshes/wheel_right_link.STL"/>
       </geometry>
     </visual>
   </link>
   <joint name="wheel_right_joint" type="continuous">
-    <origin xyz="0 -0.0701101849418637 0" rpy="0 0 0" />
-    <parent link="base_link" />
-    <child link="wheel_right_link" />
-    <axis xyz="0 1 0" />
+    <parent link="base_link"/>
+    <child link="wheel_right_link"/>
+    <axis xyz="0 1 0"/>
+    <origin xyz="0 -0.0701101849418637 0" rpy="0 0 0"/>
   </joint>
   <link name="wheel_left_link">
     <visual>
-      <origin xyz="0 0 0" rpy="-1.57 0 0" />
+      <origin xyz="0 0.014 0" rpy="1.5708 0 3.1416"/>
       <geometry>
-        <mesh filename="package://bumperbot_description/meshes/wheel_left_link.STL" scale="0.001 0.001 0.001"/>
+        <mesh filename="package://bumperbot_description/meshes/wheel_left_link.STL"/>
       </geometry>
     </visual>
   </link>
   <joint name="wheel_left_joint" type="continuous">
-    <origin xyz="0 0.0701101849418642 0" rpy="0 0 0" />
-    <parent link="base_link" />
-    <child link="wheel_left_link" />
-    <axis xyz="0 1 0" />
+    <parent link="base_link"/>
+    <child link="wheel_left_link"/>
+    <axis xyz="0 1 0"/>
+    <origin xyz="0 0.0701101849418637 0" rpy="0 0 0"/>
   </joint>
   <link name="caster_front_link">
     <visual>
-      <origin xyz="0 0 0" rpy="0 0 0" />
+      <origin xyz="0 0 0" rpy="0 0 0"/>
       <geometry>
-        <mesh filename="package://bumperbot_description/meshes/caster_front_link.STL" scale="0.001 0.001 0.001"/>
+        <mesh filename="package://bumperbot_description/meshes/caster_front_link.STL"/>
       </geometry>
     </visual>
   </link>
   <joint name="caster_front_joint" type="fixed">
-    <origin xyz="0.04755 0 -0.0275" rpy="0 0 0" />
-    <parent link="base_link" />
-    <child link="caster_front_link" />
-    <axis xyz="0 0 0" />
-  </joint>
-  <link name="caster_rear_link">
-    <visual>
-      <origin xyz="0 0 0" rpy="0 0 0" />
-      <geometry>
-        <mesh filename="package://bumperbot_description/meshes/caster_rear_link.STL" scale="0.001 0.001 0.001"/>
-      </geometry>
-    </visual>
-  </link>
-  <joint name="caster_rear_joint" type="fixed">
-    <origin xyz="-0.04755 0 -0.0275" rpy="0 0 0" />
-    <parent link="base_link" />
-    <child link="caster_rear_link" />
-    <axis xyz="0 0 0" />
+    <parent link="base_link"/>
+    <child link="caster_front_link"/>
+    <axis xyz="0 1 0"/>
+    <origin xyz="-0.04755 0 -0.0275" rpy="0 0 0"/>
   </joint>
 </robot>

File: src/bumperbot_description/urdf/bumperbot.xacro (robot description, xacro)
@@ -1,73 +1,45 @@
 <?xml version="1.0"?>
 <robot name="bumperbot" xmlns:xacro="http://ros.org/wiki/xacro">
-    <link name="base_footprint"/>
-    <link name="base_link">
-        <visual>
-            <origin xyz="0 0 0" rpy="0 0 0"/>
-            <geometry>
-                <mesh filename="package://bumperbot_description/meshes/sasi.STL" scale="0.001 0.001 0.001"/>
-            </geometry>
-        </visual>
-    </link>
-    <joint name="base_joint" type="fixed">
-        <parent link="base_footprint"/>
-        <child link="base_link"/>
-        <origin xyz="0 0 0" rpy="0 0 0.033"/>
-    </joint>
+  <link name="base_footprint"/>
+  <link name="base_link">
+    <visual>
+      <origin xyz="0 0 0" rpy="0 0 0"/>
+      <geometry>
+        <mesh filename="package://bumperbot_description/meshes/sasi.STL" scale="0.001 0.001 0.001"/>
+      </geometry>
+    </visual>
+  </link>
+  <joint name="base_joint" type="fixed">
+    <parent link="base_footprint"/>
+    <child link="base_link"/>
+    <origin xyz="0 0 0.033" rpy="0 0 0"/>
+  </joint>
   <link name="wheel_right_link">
     <visual>
-      <origin xyz="0 0 0" rpy="1.57 0 0" />
+      <origin xyz="0 -0.014 0" rpy="1.5708 0 0"/>
       <geometry>
-        <mesh filename="package://bumperbot_description/meshes/wheel_right_link.STL" scale="0.001 0.001 0.001"/>
+        <mesh filename="package://bumperbot_description/meshes/wheel_right_link.STL"/>
       </geometry>
     </visual>
   </link>
   <joint name="wheel_right_joint" type="continuous">
-    <origin xyz="0 -0.0701101849418637 0" rpy="0 0 0" />
-    <parent link="base_link" />
-    <child link="wheel_right_link" />
-    <axis xyz="0 1 0" />
+    <parent link="base_link"/>
+    <child link="wheel_right_link"/>
+    <axis xyz="0 1 0"/>
+    <origin xyz="0 -0.0701101849418637 0" rpy="0 0 0"/>
   </joint>
   <link name="wheel_left_link">
     <visual>
-      <origin xyz="0 0 0" rpy="-1.57 0 0" />
+      <origin xyz="0 0.014 0" rpy="1.5708 0 3.1416"/>
       <geometry>
-        <mesh filename="package://bumperbot_description/meshes/wheel_left_link.STL" scale="0.001 0.001 0.001"/>
+        <mesh filename="package://bumperbot_description/meshes/wheel_left_link.STL"/>
       </geometry>
     </visual>
   </link>
   <joint name="wheel_left_joint" type="continuous">
-    <origin xyz="0 0.0701101849418642 0" rpy="0 0 0" />
-    <parent link="base_link" />
-    <child link="wheel_left_link" />
-    <axis xyz="0 1 0" />
-  </joint>
-  <link name="caster_front_link">
-    <visual>
-      <origin xyz="0 0 0" rpy="0 0 0" />
-      <geometry>
-        <mesh filename="package://bumperbot_description/meshes/caster_front_link.STL" scale="0.001 0.001 0.001"/>
-      </geometry>
-    </visual>
-  </link>
-  <joint name="caster_front_joint" type="fixed">
-    <origin xyz="0.04755 0 -0.0275" rpy="0 0 0" />
-    <parent link="base_link" />
-    <child link="caster_front_link" />
-    <axis xyz="0 0 0" />
-  </joint>
-  <link name="caster_rear_link">
-    <visual>
-      <origin xyz="0 0 0" rpy="0 0 0" />
-      <geometry>
-        <mesh filename="package://bumperbot_description/meshes/caster_rear_link.STL" scale="0.001 0.001 0.001"/>
-      </geometry>
-    </visual>
-  </link>
-  <joint name="caster_rear_joint" type="fixed">
-    <origin xyz="-0.04755 0 -0.0275" rpy="0 0 0" />
-    <parent link="base_link" />
-    <child link="caster_rear_link" />
-    <axis xyz="0 0 0" />
+    <parent link="base_link"/>
+    <child link="wheel_left_link"/>
+    <axis xyz="0 1 0"/>
+    <origin xyz="0 0.0701101849418637 0" rpy="0 0 0"/>
   </joint>
 </robot>

Commit message: caster-wheel updated

File: install/bumperbot_description/share/bumperbot_description/urdf/bumperbot.xacro (robot description, xacro)
@@ -43,17 +43,16 @@
     <origin xyz="0 0.0701101849418637 0" rpy="0 0 0"/>
   </joint>
-  <link name="caster_front_link">
+  <link name="caster_wheel_link">
     <visual>
       <origin xyz="0 0 0" rpy="0 0 0"/>
       <geometry>
-        <mesh filename="package://bumperbot_description/meshes/caster_front_link.STL"/>
+        <mesh filename="package://bumperbot_description/meshes/casterwheel.STL" scale="0.0015 0.0015 0.0015"/>
       </geometry>
     </visual>
   </link>
-  <joint name="caster_front_joint" type="fixed">
+  <joint name="caster_wheel_joint" type="fixed">
     <parent link="base_link"/>
-    <child link="caster_front_link"/>
-    <axis xyz="0 1 0"/>
-    <origin xyz="-0.04755 0 -0.0275" rpy="0 0 0"/>
+    <child link="caster_wheel_link"/>
+    <origin xyz="-0.092 0 0.010" rpy="0 0 0"/>
   </joint>
 </robot>

File: src/bumperbot_description/urdf/bumperbot.xacro (robot description, xacro)
@@ -43,3 +43,16 @@
     <origin xyz="0 0.0701101849418637 0" rpy="0 0 0"/>
   </joint>
+  <link name="caster_wheel_link">
+    <visual>
+      <origin xyz="0 0 0" rpy="0 0 0"/>
+      <geometry>
+        <mesh filename="package://bumperbot_description/meshes/casterwheel.STL" scale="0.0015 0.0015 0.0015"/>
+      </geometry>
+    </visual>
+  </link>
+  <joint name="caster_wheel_joint" type="fixed">
+    <parent link="base_link"/>
+    <child link="caster_wheel_link"/>
+    <origin xyz="-0.092 0 0.010" rpy="0 0 0"/>
+  </joint>
 </robot>

Commit message: detailed

File: install/bumperbot_description/share/bumperbot_description/urdf/bumperbot.xacro (robot description, xacro)
@@ -17,5 +17,5 @@
   <link name="wheel_right_link">
     <visual>
-      <origin xyz="0 -0.014 0" rpy="1.5708 0 0"/>
+      <origin xyz="0 0 0" rpy="1.5708 0 0"/>
       <geometry>
         <mesh filename="package://bumperbot_description/meshes/wheel_right_link.STL"/>
@@ -26,5 +26,5 @@
     <parent link="base_link"/>
     <child link="wheel_right_link"/>
-    <axis xyz="0 1 0"/>
+    <axis xyz="0 1 0"/>  #Y ekseni etrafında döner
     <origin xyz="0 -0.0701101849418637 0" rpy="0 0 0"/>
   </joint>

File: src/bumperbot_description/urdf/bumperbot.xacro (robot description, xacro)
@@ -15,18 +15,24 @@
     <origin xyz="0 0 0.033" rpy="0 0 0"/>
   </joint>
-  <link name="wheel_right_link">
-    <visual>
-      <origin xyz="0 -0.014 0" rpy="1.5708 0 0"/>
-      <geometry>
-        <mesh filename="package://bumperbot_description/meshes/wheel_right_link.STL"/>
-      </geometry>
-    </visual>
-  </link>
-  <joint name="wheel_right_joint" type="continuous">
-    <parent link="base_link"/>
-    <child link="wheel_right_link"/>
-    <axis xyz="0 1 0"/>
-    <origin xyz="0 -0.0701101849418637 0" rpy="0 0 0"/>
-  </joint>
+<link name="wheel_right_link">
+  <visual>
+    <!-- STL'nin link merkezine göre hizalanması (robot konumu değil) -->
+    <origin xyz="0 -0.014 0" rpy="1.5708 0 0"/>
+    <geometry>
+      <!-- Sağ tekerin 3D modeli -->
+      <mesh filename="package://bumperbot_description/meshes/wheel_right_link.STL"/>
+    </geometry>
+  </visual>
+</link>
+<joint name="wheel_right_joint" type="continuous">
+  <!-- Tekerin bağlı olduğu ana gövde -->
+  <parent link="base_link"/>
+  <!-- Bu joint'in hareket ettirdiği parça -->
+  <child link="wheel_right_link"/>
+  <!-- Tekerin döndüğü eksen (Y ekseni) -->
+  <axis xyz="0 1 0"/>
+  <!-- Tekerin base_link'e göre robot üzerindeki konumu -->
+  <origin xyz="0 -0.07011 0" rpy="0 0 0"/>
+</joint>
   <link name="wheel_left_link">
     <visual>

Commit message: launch

File: install/bumperbot_description/share/bumperbot_description/urdf/bumperbot.xacro (robot description, xacro)
@@ -15,18 +15,24 @@
     <origin xyz="0 0 0.033" rpy="0 0 0"/>
   </joint>
-  <link name="wheel_right_link">
-    <visual>
-      <origin xyz="0 0 0" rpy="1.5708 0 0"/>
-      <geometry>
-        <mesh filename="package://bumperbot_description/meshes/wheel_right_link.STL"/>
-      </geometry>
-    </visual>
-  </link>
-  <joint name="wheel_right_joint" type="continuous">
-    <parent link="base_link"/>
-    <child link="wheel_right_link"/>
-    <axis xyz="0 1 0"/>  #Y ekseni etrafında döner
-    <origin xyz="0 -0.0701101849418637 0" rpy="0 0 0"/>
-  </joint>
+<link name="wheel_right_link">
+  <visual>
+    <!-- STL'nin link merkezine göre hizalanması (robot konumu değil) -->
+    <origin xyz="0 -0.014 0" rpy="1.5708 0 0"/>
+    <geometry>
+      <!-- Sağ tekerin 3D modeli -->
+      <mesh filename="package://bumperbot_description/meshes/wheel_right_link.STL"/>
+    </geometry>
+  </visual>
+</link>
+<joint name="wheel_right_joint" type="continuous">
+  <!-- Tekerin bağlı olduğu ana gövde -->
+  <parent link="base_link"/>
+  <!-- Bu joint'in hareket ettirdiği parça -->
+  <child link="wheel_right_link"/>
+  <!-- Tekerin döndüğü eksen (Y ekseni) -->
+  <axis xyz="0 1 0"/>
+  <!-- Tekerin base_link'e göre robot üzerindeki konumu -->
+  <origin xyz="0 -0.07011 0" rpy="0 0 0"/>
+</joint>
   <link name="wheel_left_link">
     <visual>

Commit message: en zor olanı

File: install/bumperbot_description/share/bumperbot_description/urdf/bumperbot.xacro (robot description, xacro)
@@ -1,64 +1 @@
-<?xml version="1.0"?>
-<robot name="bumperbot" xmlns:xacro="http://ros.org/wiki/xacro">
-  <link name="base_footprint"/>
-  <link name="base_link">
-    <visual>
-      <origin xyz="0 0 0" rpy="0 0 0"/>
-      <geometry>
-        <mesh filename="package://bumperbot_description/meshes/sasi.STL" scale="0.001 0.001 0.001"/>
-      </geometry>
-    </visual>
-  </link>
-  <joint name="base_joint" type="fixed">
-    <parent link="base_footprint"/>
-    <child link="base_link"/>
-    <origin xyz="0 0 0.033" rpy="0 0 0"/>
-  </joint>
-<link name="wheel_right_link">
-  <visual>
-    <!-- STL'nin link merkezine göre hizalanması (robot konumu değil) -->
-    <origin xyz="0 -0.014 0" rpy="1.5708 0 0"/>
-    <geometry>
-      <!-- Sağ tekerin 3D modeli -->
-      <mesh filename="package://bumperbot_description/meshes/wheel_right_link.STL"/>
-    </geometry>
-  </visual>
-</link>
-<joint name="wheel_right_joint" type="continuous">
-  <!-- Tekerin bağlı olduğu ana gövde -->
-  <parent link="base_link"/>
-  <!-- Bu joint'in hareket ettirdiği parça -->
-  <child link="wheel_right_link"/>
-  <!-- Tekerin döndüğü eksen (Y ekseni) -->
-  <axis xyz="0 1 0"/>
-  <!-- Tekerin base_link'e göre robot üzerindeki konumu -->
-  <origin xyz="0 -0.07011 0" rpy="0 0 0"/>
-</joint>
-  <link name="wheel_left_link">
-    <visual>
-      <origin xyz="0 0.014 0" rpy="1.5708 0 3.1416"/>
-      <geometry>
-        <mesh filename="package://bumperbot_description/meshes/wheel_left_link.STL"/>
-      </geometry>
-    </visual>
-  </link>
-  <joint name="wheel_left_joint" type="continuous">
-    <parent link="base_link"/>
-    <child link="wheel_left_link"/>
-    <axis xyz="0 1 0"/>
-    <origin xyz="0 0.0701101849418637 0" rpy="0 0 0"/>
-  </joint>
-  <link name="caster_wheel_link">
-    <visual>
-      <origin xyz="0 0 0" rpy="0 0 0"/>
-      <geometry>
-        <mesh filename="package://bumperbot_description/meshes/casterwheel.STL" scale="0.0015 0.0015 0.0015"/>
-      </geometry>
-    </visual>
-  </link>
-  <joint name="caster_wheel_joint" type="fixed">
-    <parent link="base_link"/>
-    <child link="caster_wheel_link"/>
-    <origin xyz="-0.092 0 0.010" rpy="0 0 0"/>
-  </joint>
-</robot>
+/home/saul/bumperbot_ws/src/bumperbot_description/urdf/bumperbot.xacro

File: src/bumperbot_description/urdf/bumperbot.xacro (robot description, xacro)
@@ -1,4 +1,5 @@
 <?xml version="1.0"?>
 <robot name="bumperbot" xmlns:xacro="http://ros.org/wiki/xacro">
+  <xacro:include filename="$(find bumperbot_description)/urdf/bumperbot_gazebo.xacro"/>
   <!-- Base Footprint Link -->
   <link name="base_footprint"/>

File: src/bumperbot_description/urdf/bumperbot_gazebo.xacro (robot description, xacro)
@@ -1,2 +1,29 @@
 <?xml version="1.0"?>
-<robot name="">
+<robot name="bumperbot" xmlns:xacro="http://ros.org/wiki/xacro">
+  <gazebo reference="wheel_left_link">
+    <mu1>1000000000000000.0</mu1>
+    <mu2>1000000000000000.0</mu2>
+    <kp>1000000000000.0</kp>
+    <kd>10.0</kd>
+    <minDepth>0.001</minDepth>
+    <maxVel>0.1</maxVel>
+    <fdir1>1 0 0</fdir1>
+  </gazebo>
+  <gazebo reference="wheel_right_link">
+    <mu1>1000000000000000.0</mu1>
+    <mu2>1000000000000000.0</mu2>
+    <kp>1000000000000.0</kp>
+    <kd>10.0</kd>
+    <minDepth>0.001</minDepth>
+    <maxVel>0.1</maxVel>
+    <fdir1>1 0 0</fdir1>
+  </gazebo>
+  <gazebo reference="caster_wheel_link">
+    <mu1>0.1</mu1>
+    <mu2>0.1</mu2>
+    <kp>1000000.0</kp>
+    <kd>100.0</kd>
+    <minDepth>0.001</minDepth>
+    <maxVel>1.0</maxVel>
+  </gazebo>
+</robot>
