Commit message: hatalı ama olsun düzelticem

File: install/bumperbot_description/share/bumperbot_description/urdf/bumperbot.xacro (robot description, xacro)
@@ -1 +1,109 @@
-/home/saul/bumperbot_ws/src/bumperbot_description/urdf/bumperbot.xacro
+<?xml version="1.0"?>
+<robot name="bumperbot" xmlns:xacro="http://ros.org/wiki/xacro">
+  <xacro:arg name="is_ignition" default="true"/>
+  <xacro:include filename="$(find bumperbot_description)/urdf/bumperbot_gazebo.xacro"/>
+  <!-- Base Footprint Link -->
+  <link name="base_footprint"/>
+  <!-- Base Link -->
+  <link name="base_link">
+    <visual>
+      <origin xyz="0 0 0" rpy="0 0 0"/>
+      <geometry>
+        <mesh filename="package://bumperbot_description/meshes/sasi.STL" scale="0.001 0.001 0.001"/>
+      </geometry>
+    </visual>
+    <collision>
+      <origin xyz="0 0 0" rpy="0 0 0"/>
+      <geometry>
+        <mesh filename="package://bumperbot_description/meshes/sasi.STL" scale="0.001 0.001 0.001"/>
+      </geometry>
+    </collision>
+    <inertial>
+      <mass value="5.0"/>
+      <inertia ixx="0.1" ixy="0" ixz="0" iyy="0.1" iyz="0" izz="0.1"/>
+    </inertial>
+  </link>
+  <!-- Base Joint -->
+  <joint name="base_joint" type="fixed">
+    <parent link="base_footprint"/>
+    <child link="base_link"/>
+    <origin xyz="0 0 0.033" rpy="0 0 0"/>
+  </joint>
+  <!-- Right Wheel -->
+  <link name="wheel_right_link">
+    <visual>
+      <origin xyz="0 -0.014 0" rpy="1.5708 0 0"/>
+      <geometry>
+        <mesh filename="package://bumperbot_description/meshes/wheel_right_link.STL"/>
+      </geometry>
+    </visual>
+    <collision>
+      <origin xyz="0 -0.014 0" rpy="1.5708 0 0"/>
+      <geometry>
+        <mesh filename="package://bumperbot_description/meshes/wheel_right_link.STL"/>
+      </geometry>
+    </collision>
+    <inertial>
+      <mass value="1.0"/>
+      <inertia ixx="0.01" ixy="0" ixz="0" iyy="0.01" iyz="0" izz="0.01"/>
+    </inertial>
+  </link>
+  <!-- Right Wheel Joint -->
+  <joint name="wheel_right_joint" type="continuous">
+    <parent link="base_link"/>
+    <child link="wheel_right_link"/>
+    <axis xyz="0 1 0"/>
+    <origin xyz="0 -0.07011 0" rpy="0 0 0"/>
+  </joint>
+  <!-- Left Wheel -->
+  <link name="wheel_left_link">
+    <visual>
+      <origin xyz="0 0.014 0" rpy="1.5708 0 3.1416"/>
+      <geometry>
+        <mesh filename="package://bumperbot_description/meshes/wheel_left_link.STL"/>
+      </geometry>
+    </visual>
+    <collision>
+      <origin xyz="0 0.014 0" rpy="1.5708 0 3.1416"/>
+      <geometry>
+        <mesh filename="package://bumperbot_description/meshes/wheel_left_link.STL"/>
+      </geometry>
+    </collision>
+    <inertial>
+      <mass value="1.0"/>
+      <inertia ixx="0.01" ixy="0" ixz="0" iyy="0.01" iyz="0" izz="0.01"/>
+    </inertial>
+  </link>
+  <!-- Left Wheel Joint -->
+  <joint name="wheel_left_joint" type="continuous">
+    <parent link="base_link"/>
+    <child link="wheel_left_link"/>
+    <axis xyz="0 1 0"/>
+    <origin xyz="0 0.07011 0" rpy="0 0 0"/>
+  </joint>
+  <!-- Caster Wheel -->
+  <link name="caster_wheel_link">
+    <visual>
+      <origin xyz="0 0 0" rpy="0 0 0"/>
+      <geometry>
+        <mesh filename="package://bumperbot_description/meshes/casterwheel.STL" scale="0.0015 0.0015 0.0015"/>
+      </geometry>
+    </visual>
+    <collision>
+      <origin xyz="0 0 0" rpy="0 0 0"/>
+      <geometry>
+        <box size="0.03215 0.043575 0.035122"/> <!-- Caster tekerleği boyutlarına göre kutu geometrisi -->
+      </geometry>
+    </collision>
+    <inertial>
+      <mass value="0.00766"/> <!-- Kütle 7.66 g = 0.00766 kg -->
+      <inertia ixx="0.1456842" ixy="-0.004499" ixz="-0.007876" iyy="0.1154946" iyz="-0.0382781" izz="0.0921484"/>
+    </inertial>
+  </link>
+  <!-- Caster Wheel Joint -->
+  <joint name="caster_wheel_joint" type="fixed">
+    <parent link="base_link"/>
+    <child link="caster_wheel_link"/>
+    <origin xyz="-0.092 0 0.010" rpy="0 0 0"/>
+  </joint>
+</robot>

File: install/bumperbot_description/share/bumperbot_description/urdf/bumperbot_gazebo.xacro (robot description, xacro)
@@ -1 +1,45 @@
-/home/saul/bumperbot_ws/src/bumperbot_description/urdf/bumperbot_gazebo.xacro
+<?xml version="1.0"?>
+<robot name="bumperbot" xmlns:xacro="http://ros.org/wiki/xacro">
+  <!-- Wheels -->
+  <gazebo reference="wheel_left_link">
+    <mu1>1000000000000000.0</mu1>
+    <mu2>1000000000000000.0</mu2>
+    <kp>1000000000000.0</kp>
+    <kd>10.0</kd>
+    <minDepth>0.001</minDepth>
+    <maxVel>0.1</maxVel>
+    <fdir1>1 0 0</fdir1>
+  </gazebo>
+  <gazebo reference="wheel_right_link">
+    <mu1>1000000000000000.0</mu1>
+    <mu2>1000000000000000.0</mu2>
+    <kp>1000000000000.0</kp>
+    <kd>10.0</kd>
+    <minDepth>0.001</minDepth>
+    <maxVel>0.1</maxVel>
+    <fdir1>1 0 0</fdir1>
+  </gazebo>
+  <gazebo reference="caster_wheel_link">
+    <mu1>0.1</mu1>
+    <mu2>0.1</mu2>
+    <kp>1000000.0</kp>
+    <kd>100.0</kd>
+    <minDepth>0.001</minDepth>
+    <maxVel>1.0</maxVel>
+  </gazebo>
+ <!-- ROS 2 Control -->
+  <gazebo>
+    <!-- ROS 2 Humble -->
+    <xacro:if value="$(arg is_ignition)">
+      <plugin filename="ign_ros2_control-system" name="ign_ros2_control::IgnitionROS2ControlPlugin">
+        <parameters>$(find bumperbot_controller)/config/bumperbot_controllers.yaml</parameters>
+      </plugin>
+    </xacro:if>
+    <!-- ROS 2 Iron or above -->
+    <xacro:unless value="$(arg is_ignition)">
+      <plugin filename="gz_ros2_control-system" name="gz_ros2_control::GazeboSimROS2ControlPlugin">
+        <parameters>$(find bumperbot_controller)/config/bumperbot_controllers.yaml</parameters>
+      </plugin>
+    </xacro:unless>
+  </gazebo>
+</robot>

File: install/bumperbot_description/share/bumperbot_description/urdf/bumperbot_ros2_control.xacro (robot description, xacro)
@@ -1 +1,38 @@
-/home/saul/bumperbot_ws/src/bumperbot_description/urdf/bumperbot_ros2_control.xacro
+<?xml version="1.0"?>
+<robot name="bumperbot" xmlns:xacro="http://ros.org/wiki/xacro">
+  <ros2_control name="RobotSystem" type="System"> # system → tüm robot
+  # Gazebo donanım arayüzü seçiliyor (tekrar koşullu)
+    <xacro:if value="$(arg is_ignition)">
+      <hardware>
+        <plugin>ign_ros2_control/IgnitionSytem</plugin>
+      </hardware>
+    </xacro:if>
+    <xacro:unless value="$(arg is_ignition)">
+      <hardware>
+         <plugin>gz_ros2_control/GazebıSimSystem</plugin>
+      </hardware>
+    </xacro:unless>
+    <joint name="wheel_right_joint">
+      <command_interface name="velocity"> # Bu joint hızla kontrol edilecek
+        <parameter name="min">-1</parameter>
+        <parameter name="max">1</parameter>
+      </command_interface>
+      # Geri bildirim (feedback), SLAM / odometry için zorunlu
+      <state_interface name="position"/>
+      <state_interface name="velocity"/>
+    </joint>
+    <joint name="wheel_left_joint">
+       <command_interface>
+        <parameter name="min">-1</parameter>
+        <parameter name="max">1</parameter>
+       </command_interface>
+       <state_interface name="position"/>
+       <state_interface name="velocity"/>
+    </joint>
+  </ros2_control>
+</robot>
+# NEDEN AYRI DOSYA?
+# URDF temiz kalsın
+# Gerçek robotta bu dosya değiştirilecek
+# Simülasyon / gerçek donanım ayrılacak
+# Bu profesyonel ROS yaklaşımıdır.

File: src/bumperbot_description/urdf/bumperbot.xacro (robot description, xacro)
@@ -1,5 +1,5 @@
 <?xml version="1.0"?>
 <robot name="bumperbot" xmlns:xacro="http://ros.org/wiki/xacro">
-  <xacro:arg name="is_ignition" defaul="true"/>
+  <xacro:arg name="is_ignition" default="true"/>
   <xacro:include filename="$(find bumperbot_description)/urdf/bumperbot_gazebo.xacro"/>
   <!-- Base Footprint Link -->

File: src/bumperbot_description/urdf/bumperbot_gazebo.xacro (robot description, xacro)
@@ -1,4 +1,5 @@
 <?xml version="1.0"?>
 <robot name="bumperbot" xmlns:xacro="http://ros.org/wiki/xacro">
+  <!-- Wheels -->
   <gazebo reference="wheel_left_link">
     <mu1>1000000000000000.0</mu1>
@@ -27,17 +28,18 @@
     <maxVel>1.0</maxVel>
   </gazebo>
+ <!-- ROS 2 Control -->
   <gazebo>
+    <!-- ROS 2 Humble -->
     <xacro:if value="$(arg is_ignition)">
       <plugin filename="ign_ros2_control-system" name="ign_ros2_control::IgnitionROS2ControlPlugin">
-      <parameters>$(find bumperbot_controller)/config/bumperbot_controller.yaml</parameters>
+        <parameters>$(find bumperbot_controller)/config/bumperbot_controllers.yaml</parameters>
       </plugin>
     </xacro:if>
-    # Gazebo’ya diyor ki: Benim motorlarımı ROS2 Control yönetecek
+    <!-- ROS 2 Iron or above -->
     <xacro:unless value="$(arg is_ignition)">
       <plugin filename="gz_ros2_control-system" name="gz_ros2_control::GazeboSimROS2ControlPlugin">
-      <parameters>$(find bumperbot_controller)/config/bumperbot_controller.yaml</parameters>
+        <parameters>$(find bumperbot_controller)/config/bumperbot_controllers.yaml</parameters>
       </plugin>
-    <xacro:unless>
-    # Aynı iş ama farklı plugin
+    </xacro:unless>
   </gazebo>
 </robot>
